Commit message: clean the build files

File: mower_ws/src/mower_description/urdf/mower.urdf (robot description, URDF)
Before this commit: robot mower, 3 links, 2 joints
Joints:
- joint left_wheel_joint: origin xyz=0 0.2 0 -> xyz=0 0.2 0.1 rpy=0 0 0
- joint right_wheel_joint: origin xyz=0 -0.2 0 -> xyz=0 -0.2 0.1 rpy=0 0 0
